File: Hardware/freesoc_sparkfun.brd (EAGLE design)
At the start: 160 x 100 mm, 82 parts, among them J1 5.5x2.1mm Barrel, U1 CY8C5888AXI-LP096, U2 AP2202-ADJ, U3 AP2202-ADJ, U4 AP2202-ADJ, U5 AP2202-ADJ, U6 AP2202-ADJ, U7 CY8C5868LTI-LP039

Commit message: Add some bypass caps
Parts:
- added C18: 2.2uF, SparkFun-Capacitors:0603-CAP
- added C19, C20: 1.0uF, SparkFun-Capacitors:0603-CAP
- added C21, C22, C23, C25, C27, C29, C31: 0.1uF, SparkFun-Capacitors:0402-CAP
- C13, C15: device SparkFun-Capacitors:0603-CAP -> SparkFun-Capacitors:0402-CAP
- moved S2 472.2 mm to (73.7, 15.2)
- moved S1 471.0 mm to (40.6, 41.9)
- moved JP16 453.2 mm to (10.2, 54.6)
- moved JP15 444.6 mm to (26.7, 49.5)
- moved JP17 438.0 mm to (45.7, 16.5)
- moved JP14 432.3 mm to (43.2, 35.6), turned to 180 degrees
- moved R19 425.0 mm to (15.2, 40.6), turned to 180 degrees
- moved JP18 424.7 mm to (36.8, 1.27)
- moved JP13 420.3 mm to (85.1, 29.2), turned to 270 degrees
- moved R18 420.2 mm to (15.2, 39.4), turned to 180 degrees
- moved C17 412.0 mm to (28.3, 40.9), turned to 90 degrees
- moved R20 408.9 mm to (27.9, -25.4)
- moved R21 408.9 mm to (27.9, -29.2)
- moved D5 408.9 mm to (30.5, -14.0)
- moved D6 408.9 mm to (26.7, -14.0)
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Connections:
- net N$1 renamed VCCA
- net N$10 renamed SW4
- net N$11 renamed SW3
- net N$12 renamed SW2
- net N$2 renamed ADJ2
- net N$20 renamed ADJ6
- net N$21 renamed SW6
- net N$4 renamed ADJ3
- net N$5 renamed ADJ4
- net N$7 renamed VCCD
- net N$8 renamed ADJ5
- net N$9 renamed SW5
- net GND: now also C18.2, C19.2, C20.2, C21.2, C22.2, C23.2, C25.2, C27.2, C29.2, C31.2, J1.GND
- net VDDD/VDDA: now also C18.1, C19.1, C20.1, C21.1, C22.1, C23.1, C25.1, C27.1, C31.1
- net VDDIO_1: now also C29.1
Other:
- board size 160 x 100 mm -> 116.8 x 55.9 mm

Commit message: Routed, ready for review.
Parts:
- removed JP16, JP18: (no value), SparkFun-Connectors:1X04
- removed R1, R10, R13, R4, R7: 5.62k, SparkFun-Resistors:0603-RES
- removed R11, R14, R2, R5, R8: 3.40k, SparkFun-Resistors:0603-RES
- removed R12, R15, R3, R6, R9: 4.12k, SparkFun-Resistors:0603-RES
- removed SJ3: JUMPER-PAD-2-NC_BY_TRACE, SparkFun-Passives:PAD-JUMPER-2-NC_BY_TRACE_YES_SILK
- removed SJ4, SJ5: JUMPER-PAD-2-NOYES_SILK, SparkFun-Passives:PAD-JUMPER-2-NO_YES_SILK
- removed U$1: 4-POS-DIP, SparkFun-Electromechanical:4-POS-DIP-SMD
- removed U4, U5, U6: AP2202-ADJ, SparkFun-PowerIC:SOT23-5
- added C24: 22pF, SparkFun-Capacitors:0603-CAP
- added C26, C28: 2.2uF, SparkFun-Capacitors:0603-CAP
- added S3, S4: (no value), SparkFun-Electromechanical:SWITCH-SPDT
- added Y1: 32.768kHz, SparkFun-FreqCtrl:TC26H
- added Y2: (no value), SparkFun-FreqCtrl:HC49US
- C1, C11, C16, C17, C19, C2, C20, C3, C4, C5, C6, C7, C9: device SparkFun-Capacitors:0603-CAP -> SparkFun-Capacitors:0402-CAP
- C10, C8: value 2.2uF -> 470pF
- C12, C14: value 2.2uF -> (none); device SparkFun-Capacitors:0603-CAP -> SparkFun-Capacitors:CAP-PTH-SMALL
- C18: value 2.2uF -> 22pF
- J1: value 5.5x2.1mm Barrel -> POWER_JACKPTH; device SparkFun-Connectors:POWER_JACK_SMD -> SparkFun-Connectors:POWER_JACK_PTH
- JP1, JP2: value USBSMD -> MicroB; device SparkFun-Connectors:USB-MINIB -> SparkFun-Connectors:USB-B-MICRO-SMD_V03
- JP10, JP11, JP12, JP15, JP8, JP9: value M06X2FEMALE-SMT -> 2X6 FEMALE; device SparkFun-Connectors:2X6_SMD -> SparkFun-Connectors:2X6
- JP13: device SparkFun-Connectors:2X3_SMT_POSTS -> SparkFun-Connectors:2X3
- JP4: device SparkFun-Connectors:1X06_SMD_STRAIGHT_COMBO -> SparkFun-Connectors:1X06_NO_SILK
- JP5, JP6: device SparkFun-Connectors:1X08_SMD_COMBINED -> SparkFun-Connectors:1X08_NO_SILK
- JP7: value M10SMD_COMBO-FEMALE -> M10NO_SILK_PTH_FEMALE; device SparkFun-Connectors:1X10_SMD_COMBINED -> SparkFun-Connectors:1X10_NO_SILK
- U1: value CY8C5888AXI-LP096 -> CY8C5868AXI-LP035
- U2: value AP2202-ADJ -> MIC5219 5V
- U3: value AP2202-ADJ -> MIC5219 3.3V
- moved R21 76.1 mm to (47.0, 44.5), turned to 90 degrees
- moved D5 63.8 mm to (47.0, 47.6)
- moved R20 57.8 mm to (19.1, 31.8), turned to 90 degrees
- moved C18 55.9 mm to (76.2, 20.3), turned to 0 degrees
- moved D6 50.1 mm to (19.1, 35.6)
- moved C12 43.7 mm to (70.5, 10.2), turned to 0 degrees
- moved S1 36.1 mm to (6.35, 30.5), turned to 180 degrees
- moved C14 33.8 mm to (56.5, 10.2)
- moved JP10 25.0 mm to (101.6, 3.81), turned to 180 degrees
- moved C6 19.9 mm to (72.4, 28.8), turned to 0 degrees
- moved C4 18.6 mm to (60.1, 15.2), turned to 270 degrees
- moved JP8 18.0 mm to (109.2, 38.1), turned to 90 degrees
- moved C5 17.8 mm to (72.4, 27.6), turned to 0 degrees
- moved C2 17.7 mm to (60.8, 40.3), turned to 0 degrees
- moved JP14 16.9 mm to (39.4, 19.1), turned to 90 degrees
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Connections:
- net N$18 renamed PSOC_D+_PAD
- net N$19 renamed DEBUG_D-_PAD
- net N$22 renamed DEBUG_D+_PAD
- net N$3 renamed PSOC_D-_PAD
- removed net ADJ2: R1.2, R2.1, R3.1, U2.4
- removed net ADJ3: R4.2, R5.1, R6.1, U3.4
- removed net ADJ4: R7.2, R8.1, R9.1, U4.4
- removed net ADJ5: R10.2, R11.1, R12.1, U5.4
- removed net ADJ6: R13.2, R14.1, R15.1, U6.4
- removed net DEBUG_D+: JP2.D+, R18.2
- removed net DEBUG_D-: JP2.D-, R19.2
- removed net N$24: R20.1
- removed net N$31: SJ4.1, U7.38
- removed net N$32: SJ5.1, U7.39
- removed net PSOC_D+: JP1.D+, R16.2
- removed net PSOC_D-: JP1.D-, R17.2
- removed net SW2: R3.2, U$1.4
- removed net SW3: R6.2, U$1.3
- removed net SW4: R9.2, U$1.2
- removed net SW5: R12.2, U$1.1
- removed net SW6: R15.2, SJ3.1
- removed net VDDD/VDDA: C18.1, C19.1, C2.1, C20.1, C21.1, C22.1, C23.1, C25.1, C27.1, C3.1, C31.1, C4.1, C5.1, C6.1, JP14.1, JP15.10, JP15.9, JP16.2, JP6.4, JP6.5, R13.1, U1.37, U1.65, U1.88, U6.5, U7.17, U7.24, U7.44, U7.52, U7.59, U7.67
- removed net VDDIO_0: C14.1, C15.1, JP8.10, JP8.9, JP9.10, JP9.9, R10.1, U1.75, U5.5
- removed net VDDIO_1: C12.1, C13.1, C29.1, JP10.10, JP10.9, JP11.10, JP11.9, JP17.1, R7.1, U1.26, U4.5, U7.35
- removed net VDDIO_2: C10.1, C11.1, JP13.2, JP6.7, R4.1, U1.100, U3.5
- removed net VDDIO_3: C8.1, C9.1, JP12.10, JP12.9, JP18.2, R1.1, U1.50, U2.5
- new net 3.3V: C26.2, JP6.5, S3.3, S4.3, U3.5
- new net 5V: C20.1, C23.1, C28.2, C5.1, C6.1, JP6.4, S3.1, S4.1, U1.65, U2.5, U7.44
- new net DEBUG_D+_BUS: JP2.D+1, R18.2
- new net DEBUG_D-_BUS: JP2.D-1, R19.2
- new net DEBUG_LED: R20.1, U7.62
- new net N$1: C8.1, U3.4
- new net N$2: C10.1, U2.4
- new net PSOC_D+_BUS: JP1.D+1, R16.2
- new net PSOC_D-_BUS: JP1.D-1, R17.2
- new net VDDIO: C13.1, C15.1, C19.1, C2.1, C21.1, C22.1, C25.1, C27.1, C29.1, C3.1, C31.1, C4.1, C9.1, JP10.10, JP10.9, JP11.10, JP11.9, JP12.10, JP12.9, JP14.1, JP15.10, JP15.9, JP17.1, JP8.10, JP8.9, JP9.10, JP9.9, S4.2, U1.26, U1.37, U1.50, U1.75, U1.88, U7.17, U7.24, U7.35, U7.52, U7.59, U7.67
- new net VDDIO_ARDUINO: C11.1, JP13.2, JP6.7, S3.2, U1.100
- net A0: now also U1.94; no longer U1.89
- net A1: now also U1.93; no longer U1.90
- net A2: now also U1.92; no longer U1.91
- net A3: now also U1.91; no longer U1.92
- net A4: now also JP7.10, U1.90; no longer JP7.10A, JP7.10B, U1.93
- net A5: now also JP7.9, U1.89; no longer JP7.9A, JP7.9B, U1.94
- net AGND: now also C17.2, C20.2, C23.2, U7.43
- net D0: now also U1.95; no longer U1.99
- net D1: now also U1.96; no longer U1.1
- net D10: now also JP7.3, U1.6; no longer JP7.3A, JP7.3B, U1.2
- net D11: now also JP7.4, U1.7; no longer JP7.4A, JP7.4B, U1.8
- net D12: now also JP7.5, U1.8; no longer JP7.5A, JP7.5B, U1.7
- net D13: now also JP7.6; no longer JP7.6A, JP7.6B
- net D2: now also U1.97; no longer U1.98
- net D3: now also U1.98; no longer U1.5
- net D4: now also U1.99; no longer U1.95
- net D5: now also U1.1; no longer U1.6
- net D6: now also U1.2; no longer U1.3
- net D7: now also U1.3; no longer U1.97
- net D8: now also JP7.1, U1.4; no longer JP7.1A, JP7.1B, U1.96
- net D9: now also JP7.2, U1.5; no longer JP7.2A, JP7.2B, U1.4
- net DEBUG_I2C0_SCL: no longer JP16.4
- net DEBUG_I2C0_SDA: no longer JP16.3
- net GND: now also C24.2, C26.1, C28.1, J1.GNDBREAK, JP1.GND1, JP1.SHIELD1, JP1.SHIELD2, JP1.SHIELD3, JP2.GND1, JP2.SHIELD1, JP2.SHIELD2, JP2.SHIELD3, JP7.7; no longer C17.2, C20.2, C23.2, J1.P$4, JP1.GND, JP16.1, JP18.1, JP2.GND, JP7.7A, JP7.7B, R11.2, R14.2, R2.2, R5.2, R8.2, SJ3.2, U$1.5, U$1.6, U$1.7, U$1.8, U4.2, U5.2, U6.2, U7.43
- net N$13: now also J1.PWR; no longer J1.VIN0
- net N$15: now also JP1.VBUS1; no longer JP1.VBUS
- net P12.0: no longer JP18.4, SJ4.2
- net P12.1: no longer JP18.3, SJ5.2
- net P15.0: now also C14.1, Y2.1
- net P15.1: now also C12.1, Y2.2
- net P15.2: now also C18.1, Y1.2
- net P15.3: now also C24.1, Y1.1
- net P4.0: now also JP9.2; no longer JP9.1
- net P4.1: now also JP9.1; no longer JP9.2
- net P4.2: now also JP9.4; no longer JP9.3
- net P4.3: now also JP9.3; no longer JP9.4
- net P4.4: now also JP9.6; no longer JP9.5
- net P4.5: now also JP9.5; no longer JP9.6
- net P4.6: now also JP9.8; no longer JP9.7
- net P4.7: now also JP9.7; no longer JP9.8
- net P5.0: now also JP11.2; no longer JP11.1
- net P5.1: now also JP11.1; no longer JP11.2
- net P5.2: now also JP11.4; no longer JP11.3
- net P5.3: now also JP11.3; no longer JP11.4
- net P5.4: now also JP11.6; no longer JP11.5
- net P5.5: now also JP11.5; no longer JP11.6
- net P5.6: now also JP11.8; no longer JP11.7
- net P5.7: now also JP11.7; no longer JP11.8
- net V_DEBUG: now also JP2.VBUS1; no longer JP2.VBUS
- net V_IN: no longer U4.1, U4.3, U5.1, U5.3, U6.1, U6.3
Routing:
- net VDDIO_ARDUINO: track 0.00 -> 136.8 mm, vias 0 -> 1
- net P1.1: track 0.00 -> 134.1 mm, vias 0 -> 3
- net 5V: track 0.00 -> 131.4 mm, vias 0 -> 2
- net P1.3: track 0.00 -> 126.1 mm, vias 0 -> 3
- net !RESET: track 0.00 -> 125.0 mm, vias 0 -> 7
- net P1.4: track 0.00 -> 120.3 mm, vias 0 -> 3
- net P1.0: track 0.00 -> 112.0 mm, vias 0 -> 2
- net V_IN: track 0.00 -> 111.4 mm
- net GND: track 0.00 -> 97.7 mm, vias 0 -> 40
- net PSOC_D+_PAD: track 0.00 -> 93.5 mm, vias 0 -> 2
- net PSOC_D-_PAD: track 0.00 -> 93.3 mm, vias 0 -> 2
- net A4: track 0.00 -> 92.4 mm, vias 0 -> 4
- net A5: track 0.00 -> 88.8 mm, vias 0 -> 4
- net P1.2: track 0.00 -> 73.4 mm, vias 0 -> 1
- net P1.7: track 0.00 -> 68.6 mm, vias 0 -> 1
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- added copper zone on layer 1, net AGND
- added copper zone on layer 16, net AGND
- added copper zone on layer 1, net GND
- added copper zone on layer 15, net GND
- added copper zone on layer 1, net VDDIO
- added copper zone on layer 16, net VDDIO
- added copper zone on layer 2, net VDDIO
Other:
- board size 116.8 x 55.9 mm -> 110.5 x 53.3 mm

Commit message: Routed, with board checklist.
Parts:
- removed PT1: 2PT_GND_TIE, SparkFun-Passives:2PT_GND_TIE
- added C30, C32, C33, C34, C35, C36: 0.1uF, SparkFun-Capacitors:0402-CAP
- added FID1, FID2: FIDUCIAL1X2, SparkFun-Aesthetics:FIDUCIAL-1X2
- added LOGO1: SFE_LOGO_NAME_FLAME.2_INCH, SparkFun-Aesthetics:SFE_LOGO_NAME_FLAME_.2
- added LOGO2: OSHW-LOGOS, SparkFun-Aesthetics:OSHW-LOGO-S
- added S5, S6: SWITCH-MOMENTARY-2SMD, SparkFun-Electromechanical:TACTILE-SWITCH-SMD
- added SJ3, SJ4, SJ5: JUMPER-PAD-2-NO, SparkFun-Passives:PAD-JUMPER-2-NO_NO_SILK
- added STANDOFF1, STANDOFF2, STANDOFF3, STANDOFF4: STAND-OFF, SparkFun-Electromechanical:STAND-OFF
- added U$1: FOUR_LAYER_WARNING, SparkFun-Aesthetics:FOUR_LAYER_WARNING
- C4: value 0.1uF -> 1.0uF
- JP10: value 2X6 FEMALE -> (none); device SparkFun-Connectors:2X6 -> SparkFun-Connectors:1X08
- JP4: device SparkFun-Connectors:1X06_NO_SILK -> SparkFun-Connectors:1X06
- JP5, JP6: device SparkFun-Connectors:1X08_NO_SILK -> SparkFun-Connectors:1X08
- JP7: value M10NO_SILK_PTH_FEMALE -> M10SILK_FEMALE_PTH; device SparkFun-Connectors:1X10_NO_SILK -> SparkFun-Connectors:1X10
- R16, R17, R18, R19: device SparkFun-Resistors:0603-RES -> SparkFun-Resistors:0402-RES
- R20, R21: value 330 -> 1K
- SJ1: value JUMPER-PAD-2-NC_BY_TRACE -> JUMPER-PAD-2-NC_BY_PASTE; device SparkFun-Passives:PAD-JUMPER-2-NC_BY_TRACE_YES_SILK -> SparkFun-Passives:PAD-JUMPER-2-NC_BY_PASTE_YES_SILK
- moved FRAME1 172.0 mm to (20.3, -27.9)
- moved FRAME2 172.0 mm to (20.3, -27.9)
- moved FRAME3 172.0 mm to (20.3, -27.9)
- moved R16 48.7 mm to (55.9, 13.3), turned to 180 degrees
- moved R17 47.5 mm to (55.9, 12.1), turned to 180 degrees
- moved R19 28.4 mm to (35.9, 31.2), turned to 0 degrees
- moved R18 28.3 mm to (35.9, 30.1), turned to 0 degrees
- moved R20 19.0 mm to (37.7, 35.2), turned to 0 degrees
- moved D6 18.7 mm to (37.7, 36.8), turned to 90 degrees
- moved JP10 15.3 mm to (86.4, 2.54), turned to 0 degrees
- moved S3 14.2 mm to (20.3, 5.08)
- moved S4 14.2 mm to (20.3, 10.2)
- moved D5 4.84 mm to (47.4, 42.8), turned to 270 degrees
- moved D4 3.81 mm to (15.6, 49.1)
- moved SJ2 3.81 mm to (15.6, 46.2)
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Connections:
- removed net AGND: C1.2, C17.2, C20.2, C23.2, C5.2, C6.2, PT1.P$1, U1.64, U7.43
- removed net DEBUG_I2C0_SCL: U7.3
- removed net DEBUG_I2C0_SDA: U7.4
- removed net DEBUG_P0.2: JP15.3, U7.50
- removed net DEBUG_P0.3: JP15.4, U7.51
- removed net DEBUG_P0.4: JP15.5, U7.53
- removed net DEBUG_P0.5: JP15.6, U7.54
- removed net DEBUG_P0.6: JP15.7, U7.55
- removed net DEBUG_P0.7: JP15.8, U7.56
- new net DEBUG_DS_BP: C30.1, U7.51
- new net DEBUG_P1.2: JP15.2, U7.13
- new net DEBUG_P12.6: JP15.9, U7.20
- new net DEBUG_P12.7: JP15.10, U7.21
- new net DEBUG_P3.0: JP15.12, U7.29
- new net DEBUG_P3.4: JP15.5, U7.33
- new net DEBUG_P3.5: JP15.6, U7.34
- new net DEBUG_P3.6: JP15.7, U7.36
- new net DEBUG_P3.7: JP15.8, U7.37
- new net DEBUG_SAR0_BP: C33.1, U7.53
- new net DEBUG_SAR1_BP: C32.1, U7.50
- new net DEBUG_USER_BTN: S5.1, U7.18
- new net N$3: C34.1, SJ5.2
- new net N$4: C35.1, SJ4.2
- new net N$5: C36.1, SJ3.2
- net !RESET: now also U7.66; no longer U7.33
- net DEBUG_LED: now also U7.30; no longer U7.62
- net DEBUG_P0.0: now also JP15.3; no longer JP15.1
- net DEBUG_P0.1: now also JP15.4; no longer JP15.2
- net GND: now also C1.2, C17.2, C20.2, C23.2, C30.2, C32.2, C33.2, C34.2, C35.2, C36.2, C5.2, C6.2, JP10.2, S5.3, S6.3, U1.64, U7.43; no longer JP10.11, JP10.12, JP15.12, PT1.P$2
- net P0.2: now also SJ3.1
- net P0.3: now also SJ4.1
- net P0.4: now also SJ5.1
- net P1.0: now also U7.62; no longer JP10.1, U7.29
- net P1.1: now also U7.63; no longer JP10.2, U7.30
- net P1.2: now also S6.1; no longer JP10.3
- net P1.3: no longer JP10.4, U7.31
- net P1.4: no longer JP10.5, U7.32
- net P1.5: no longer JP10.6
- net P1.6: no longer JP10.7
- net P1.7: no longer JP10.8
- net P12.0: now also JP10.3
- net P12.1: now also JP10.4
- net P12.2: now also JP10.5
- net P12.3: now also JP10.6
- net P12.6: now also JP10.7
- net P12.7: now also JP10.8
- net VDDIO: now also JP10.1, JP15.1; no longer JP10.10, JP10.9, JP15.10, JP15.9
Routing:
- net P1.3: track 126.1 -> 10.3 mm, vias 3 -> 0
- net P1.4: track 120.3 -> 10.9 mm, vias 3 -> 0
- net P1.1: track 134.1 -> 46.7 mm
- net PSOC_D+_PAD: track 93.5 -> 7.36 mm, vias 2 -> 0
- net PSOC_D-_PAD: track 93.3 -> 9.21 mm, vias 2 -> 0
- net 5V: track 131.4 -> 212.3 mm, vias 2 -> 11
- net P1.0: track 112.0 -> 39.7 mm, vias 2 -> 1
- net P1.7: track 68.6 -> 0.00 mm, vias 1 -> 0
- net P1.5: track 68.5 -> 0.00 mm, vias 1 -> 0
- net P1.6: track 66.6 -> 0.00 mm, vias 1 -> 0
- net P12.7: track 0.00 -> 63.3 mm, vias 0 -> 2
- net P12.6: track 0.00 -> 61.5 mm, vias 0 -> 2
- net P12.3: track 0.00 -> 59.1 mm, vias 0 -> 2
- net P12.2: track 0.00 -> 56.9 mm, vias 0 -> 2
- net PSOC_D+_BUS: track 8.65 -> 61.1 mm, vias 0 -> 2
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- removed copper zone on layer 1, net AGND
- removed copper zone on layer 16, net AGND
- removed copper zone on layer 1, net VDDIO
- removed copper zone on layer 16, net VDDIO
Other:
- board size 110.5 x 53.3 mm -> 116.8 x 53.3 mm
- board text added: "!RESET"
- board text added: "+"
- board text added: "-"
- board text added: "0.0"
- board text added: "0.1"
- board text added: "0.2"
- board text added: "0.3"
- board text added: "0.4"
- board text added: "0.5"
- board text added: "0.6"
- board text added: "0.7"
- board text added: "1.2"
- board text added: "12.6"
- board text added: "12.7"
- board text added: "2.5V-12V"
- board text added: "3.0"
- board text added: "3.1"
- board text added: "3.2"
- board text added: "3.3"
- board text added: "3.3V"
- board text added: "3.4"
- board text added: "3.5"
- board text added: "3.6"
- board text added: "3.7"
- board text added: "4.0"
- board text added: "4.1"
- board text added: "4.2"
- board text added: "4.3"
- board text added: "4.4"
- board text added: "4.5"
- board text added: "4.6"
- board text added: "4.7"
- board text added: "5.0"
- board text added: "5.1"
- board text added: "5.2"
- board text added: "5.3"
- board text added: "5.4"
- board text added: "5.5"
- board text added: "5.6"
- board text added: "5.7"
- board text added: "5V"
- board text added: "A0 P15.5"
- board text added: "A1 P15.4"
- board text added: "A2 P6.3"
- board text added: "A3 P6.2"
- board text added: "A4/SCL P6.1"
- board text added: "A5/SDA P6.0"
- board text added: "ARDUINO"
- board text added: "BATT ISOLATE"
- board text added: "D BYPASS"
- board text added: "D0/RX P2.0"
- board text added: "D1/TX P2.1"
- board text added: "D10/CS P6.4/PWM"
- board text added: "D11/MOSI P6.5/PWM"
- board text added: "D12/MISO P6.6"
- board text added: "D13 P6.7/SCK"
- board text added: "D2/INT0 P2.2"
- board text added: "D3/INT1 P2.3/PWM"
- board text added: "D4 P2.4"
- board text added: "D5/PWM P2.5"
- board text added: "D6/PWM P2.6"
- board text added: "D7 P2.7"
- board text added: "D8 P12.4"
- board text added: "D9/PWM P12.5"
- board text added: "DEBUGGER"
- board text added: "DEBUGGER BTN P1.6"
- board text added: "DEBUGGER IO"
- board text added: "DEBUGGER LED P3.1"
- board text added: "DEBUGGER RESET"
- board text added: "DEBUGGER SWD PORT"
- board text added: "GND"
- board text added: "M. Hord"
- board text added: "PSOC"
- board text added: "SIO P12.0"
- board text added: "SIO P12.1"
- board text added: "SIO P12.2"
- board text added: "SIO P12.3"
- board text added: "SIO P12.6"
- board text added: "SIO P12.7"
- board text added: "TARGET"
- board text added: "TARGET RESET"
- board text added: "TARGET SWD PORT"
- board text added: "USER BTN P1.2"
- board text added: "USER LED D13/P6.7"
- board text added: "V SEL"
- board text added: "VDDIO"
- board text added: "VDDIO ARDUINO"
- board text added: "V_IN"
- board text added: "v01"

Commit message: Ready for QC review
Parts:
- moved S5 31.5 mm to (12.7, 35.7)
- moved D1 3.30 mm to (14.0, 24.6)
Routing:
- net DEBUG_USER_BTN: track 12.7 -> 28.9 mm, vias 2 -> 3
- net N$15: track 10.3 -> 7.41 mm
- net GND: track 121.2 -> 121.8 mm
Changed lines of the file:
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@@
 <layers>
 <layer number="1" name="Top" color="4" fill="1" visible="yes" active="yes"/>
-<layer number="2" name="Route2" color="1" fill="3" visible="no" active="yes"/>
+<layer number="2" name="Route2" color="1" fill="3" visible="yes" active="yes"/>
 <layer number="15" name="Route15" color="4" fill="6" visible="no" active="yes"/>
 <layer number="16" name="Bottom" color="1" fill="1" visible="yes" active="yes"/>
@@
 <text x="85.09" y="17.78" size="0.8128" layer="21" font="vector" ratio="15" align="center-left">TARGET
 RESET</text>
-<text x="10.922" y="32.385" size="0.8128" layer="21" font="vector" ratio="15" align="center-left">DEBUGGER
+<text x="6.096" y="26.543" size="0.8128" layer="21" font="vector" ratio="15" align="center-left">DEBUGGER
 RESET</text>
 <circle x="53.467" y="34.036" radius="0.179603125" width="0.4064" layer="21"/>
@@
 <text x="6.731" y="38.1" size="0.8128" layer="21" font="vector" ratio="15" rot="R90" align="bottom-center">DEBUGGER</text>
 <text x="7.62" y="22.86" size="0.8128" layer="21" font="vector" ratio="15" rot="R90" align="bottom-center">TARGET</text>
-<text x="41.275" y="35.56" size="0.8128" layer="21" font="vector" ratio="15" align="center-left">DEBUGGER BTN
+<text x="16.637" y="30.099" size="0.8128" layer="21" font="vector" ratio="15" rot="R90" align="center-left">DEBUGGER BTN
 P1.6</text>
 <text x="95.885" y="19.558" size="1.016" layer="21" font="vector" ratio="15">USER BTN
@@
 <attribute name="PROD_ID" value="IC-12190" x="60.96" y="26.67" size="1.778" layer="27" font="vector" ratio="15" display="off"/>
 </element>
-<element name="D1" library="SparkFun-DiscreteSemi" package="SMA-DIODE" value="MBRA140" x="13.97" y="27.94">
-<attribute name="PROD_ID" value="DIO-08053" x="13.97" y="27.94" size="1.778" layer="27" font="vector" ratio="15" display="off"/>
+<element name="D1" library="SparkFun-DiscreteSemi" package="SMA-DIODE" value="MBRA140" x="13.97" y="24.638">
+<attribute name="PROD_ID" value="DIO-08053" x="13.97" y="24.638" size="1.778" layer="27" font="vector" ratio="15" display="off"/>
 </element>
 <element name="D2" library="SparkFun-DiscreteSemi" package="SMA-DIODE" value="MBRA140" x="13.97" y="41.91">
@@
 <element name="STANDOFF3" library="SparkFun-Electromechanical" package="STAND-OFF" value="STAND-OFF" x="114.3" y="50.8"/>
 <element name="STANDOFF4" library="SparkFun-Electromechanical" package="STAND-OFF" value="STAND-OFF" x="114.3" y="2.54"/>
-<element name="S5" library="SparkFun-Electromechanical" package="TACTILE-SWITCH-SMD" value="SWITCH-MOMENTARY-2SMD" x="43.815" y="30.607" rot="R90">
-<attribute name="PROD_ID" value="SWCH-08247" x="43.815" y="30.607" size="1.778" layer="27" font="vector" ratio="15" rot="R90" display="off"/>
+<element name="S5" library="SparkFun-Electromechanical" package="TACTILE-SWITCH-SMD" value="SWITCH-MOMENTARY-2SMD" x="12.7" y="35.687" rot="R90">
+<attribute name="PROD_ID" value="SWCH-08247" x="12.7" y="35.687" size="1.778" layer="27" font="vector" ratio="15" rot="R90" display="off"/>
 </element>
 <element name="S6" library="SparkFun-Electromechanical" package="TACTILE-SWITCH-SMD" value="SWITCH-MOMENTARY-2SMD" x="100.33" y="16.51" rot="R180">
@@
 <via x="46.99" y="41.529" extent="1-16" drill="0.254"/>
 <contactref element="S5" pad="3"/>
-<wire x1="45.72" y1="27.813" x2="44.577" y2="27.813" width="0.2032" layer="1"/>
-<wire x1="44.577" y1="27.813" x2="44.45" y2="27.94" width="0.2032" layer="1"/>
-<via x="44.45" y="27.94" extent="1-16" drill="0.254"/>
 <contactref element="S6" pad="3"/>
 <wire x1="103.124" y1="18.415" x2="103.124" y2="19.304" width="0.2032" layer="1"/>
@@
 <wire x1="19.319" y1="33.543" x2="19.304" y2="33.528" width="0.2032" layer="1"/>
 <via x="19.304" y="33.528" extent="1-16" drill="0.254"/>
+<wire x1="14.605" y1="32.893" x2="12.827" y2="32.893" width="0.2032" layer="1"/>
+<wire x1="12.827" y1="32.893" x2="12.7" y2="33.02" width="0.2032" layer="1"/>
+<via x="12.7" y="33.02" extent="1-16" drill="0.254"/>
 </signal>
 <signal name="N$13">
@@
 <wire x1="5.872" y1="24.16" x2="6.35" y2="24.638" width="0.2032" layer="1"/>
 <wire x1="6.35" y1="24.638" x2="11.176" y2="24.638" width="0.762" layer="1"/>
-<wire x1="11.176" y1="24.638" x2="11.811" y2="25.273" width="0.762" layer="1"/>
-<wire x1="11.811" y1="25.273" x2="11.811" y2="27.931" width="0.762" layer="1"/>
-<wire x1="11.811" y1="27.931" x2="11.82" y2="27.94" width="0.762" layer="1"/>
+<wire x1="11.176" y1="24.638" x2="11.82" y2="24.638" width="0.254" layer="1"/>
 </signal>
 <signal name="N$16">
@@
 <contactref element="D3" pad="C"/>
 <contactref element="SJ1" pad="1"/>
-<wire x1="16.12" y1="41.91" x2="16.12" y2="27.94" width="0.762" layer="1"/>
-<wire x1="16.12" y1="27.94" x2="16.12" y2="24.257" width="0.762" layer="1"/>
+<wire x1="16.12" y1="41.91" x2="16.12" y2="24.638" width="0.762" layer="1"/>
+<wire x1="16.12" y1="24.638" x2="16.12" y2="24.257" width="0.762" layer="1"/>
 <wire x1="16.12" y1="24.257" x2="16.12" y2="23.74" width="0.762" layer="1"/>
 <wire x1="13.58" y1="17.78" x2="15.748" y2="17.78" width="0.762" layer="1"/>
@@
 <contactref element="S5" pad="1"/>
 <contactref element="U7" pad="18"/>
-<wire x1="31.84" y1="29.82" x2="32.537" y2="29.82" width="0.2032" layer="1"/>
-<wire x1="32.537" y1="29.82" x2="33.02" y2="29.337" width="0.2032" layer="1"/>
-<wire x1="33.02" y1="29.337" x2="33.02" y2="29.083" width="0.2032" layer="1"/>
-<via x="33.02" y="29.083" extent="1-16" drill="0.254"/>
-<wire x1="33.02" y1="29.083" x2="41.275" y2="29.083" width="0.2032" layer="16"/>
-<wire x1="41.275" y1="29.083" x2="41.91" y2="29.718" width="0.2032" layer="16"/>
-<via x="41.91" y="29.718" extent="1-16" drill="0.254"/>
-<wire x1="41.91" y1="29.718" x2="41.91" y2="27.813" width="0.2032" layer="1"/>
+<wire x1="31.84" y1="29.82" x2="32.41" y2="29.82" width="0.2032" layer="1"/>
+<wire x1="32.41" y1="29.82" x2="33.02" y2="29.21" width="0.2032" layer="1"/>
+<via x="33.02" y="29.21" extent="1-16" drill="0.254"/>
+<wire x1="33.02" y1="29.21" x2="31.623" y2="30.607" width="0.2032" layer="16"/>
+<wire x1="31.623" y1="30.607" x2="31.623" y2="33.02" width="0.2032" layer="16"/>
+<wire x1="31.623" y1="33.02" x2="31.242" y2="33.401" width="0.2032" layer="16"/>
+<wire x1="31.242" y1="33.401" x2="27.051" y2="33.401" width="0.2032" layer="16"/>
+<wire x1="27.051" y1="33.401" x2="26.67" y2="33.02" width="0.2032" layer="16"/>
+<wire x1="26.67" y1="33.02" x2="19.685" y2="33.02" width="0.2032" layer="16"/>
+<wire x1="19.685" y1="33.02" x2="19.05" y2="32.385" width="0.2032" layer="16"/>
+<wire x1="19.05" y1="32.385" x2="19.05" y2="31.75" width="0.2032" layer="16"/>
+<via x="19.05" y="31.75" extent="1-16" drill="0.254"/>
+<wire x1="19.05" y1="31.75" x2="12.7" y2="31.75" width="0.2032" layer="2"/>
+<via x="12.7" y="31.75" extent="1-16" drill="0.254"/>
+<wire x1="12.7" y1="31.75" x2="10.922" y2="31.75" width="0.2032" layer="1"/>
+<wire x1="10.922" y1="31.75" x2="10.795" y2="31.877" width="0.2032" layer="1"/>
+<wire x1="10.795" y1="31.877" x2="10.795" y2="32.893" width="0.2032" layer="1"/>
 </signal>
 </signals>
