File: Hardware/freesoc_sparkfun.sch (EAGLE design)
At the start: 94 parts, among them U1 CY8C5868AXI-LP035, U2 MIC5219 5V, U3 MIC5219 3.3V, U7 CY8C5868LTI-LP039, Y1 32.768kHz

Commit message: v10 almost ready
Parts:
- added C37, C38: 0.1uF, SparkFun-Capacitors:0.1UF-16V(+-10%)(0402)
- added R1, R2: 4.7K, SparkFun-Resistors:4.7KOHM-1/10W-1%(0603)
- added R3, R4: 10K, SparkFun-Resistors:10KOHM-1/10W-1%(0603)0603
- added R5, R6: 20k, SparkFun-Resistors:20KOHM1/10W1%(0603)
- FRAME1: VERSION v02 -> v10
- FRAME2, FRAME3: DESIGNER (none) -> M. Hord; VERSION (none) -> v10
- U1: value CY8C5868AXI-LP035 -> CY8C5888AXI-LP035
Connections:
- removed net DEBUG_USER_BTN: S5.1, U7G2.P1[6]
- removed net N$15: D1.A, JP1.VCC
- new net DEBUG_BTN: S5.1, U7G3.P2[2]
- new net V_BUS_DEBUG: R4.2, R5.2, U7G2.P1[6]
- new net V_BUS_HOST: R3.2, R6.2, U1G2.P1[6]
- new net V_HOST: D1.A, JP1.VCC, R3.1
- net !DEBUG_RESET: now also C38.1, R2.1
- net !RESET: now also C37.1, R1.1
- net 3.3V: now also C19.1, C2.1, C21.1, C22.1, C3.1, C4.1, R1.2, R2.2, U1G5.VDDD0, U1G5.VDDD1, U7G5.VDDD0, U7G5.VDDD1
- net GND: now also C37.2, C38.2, R5.1, R6.1
- net VDDIO: no longer C19.1, C2.1, C21.1, C22.1, C3.1, C4.1, U1G5.VDDD0, U1G5.VDDD1, U7G5.VDDD0, U7G5.VDDD1
- net V_DEBUG: now also R4.1
Other:
- note removed: "02"
- note removed: "M. Hord"
- moved on the sheet: D6, R20, S1, S2, S5
