File: Hardware/SparkFun_FreeSoC2.sch (EAGLE design)
At the start: 109 parts, among them U1 CY8C5888AXI-LP096, U2 MIC5219 5V, U3 MIC5219 3.3V, U4 2A/20V, U7 CY8C5868LTI-LP039, Y1 32.768kHz

Commit message: Fix USB port anchoring to isolate shield from ground
Connections:
- new net ANCHOR_POUR: JP1.SHIELD, JP2.SHIELD
- net GND: no longer JP1.SHIELD, JP2.SHIELD
Other:
- note added: "14"
- note removed: "13"
Changed lines of the file:
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@@
 <layer number="112" name="tSilk" color="7" fill="1" visible="yes" active="yes"/>
 <layer number="113" name="IDFDebug" color="7" fill="1" visible="yes" active="yes"/>
+<layer number="114" name="Badge_Outline" color="7" fill="1" visible="yes" active="yes"/>
+<layer number="115" name="ReferenceISLANDS" color="7" fill="1" visible="yes" active="yes"/>
 <layer number="116" name="Patch_BOT" color="9" fill="4" visible="no" active="yes"/>
 <layer number="118" name="Rect_Pads" color="7" fill="1" visible="yes" active="yes"/>
@@
 </variantdefs>
 <classes>
-<class number="0" name="signal" width="0.2032" drill="0.254">
-<clearance class="0" value="0.1524"/>
+<class number="0" name="signal" width="0.1778" drill="0.381">
+<clearance class="0" value="0.1778"/>
 </class>
 <class number="1" name="AVCC" width="0.508" drill="0.508">
-<clearance class="1" value="0.1524"/>
+<clearance class="1" value="0.1778"/>
 </class>
 <class number="2" name="ARDUINO_VCC" width="0.508" drill="0.381">
@@
 <part name="SUPPLY7" library="SparkFun-Aesthetics" deviceset="5V" device=""/>
 <part name="GND4" library="SparkFun-Aesthetics" deviceset="GND" device=""/>
-<part name="GND5" library="SparkFun-Aesthetics" deviceset="GND" device=""/>
 <part name="C12" library="SparkFun-Capacitors" deviceset="CAP" device="PTH"/>
 <part name="C14" library="SparkFun-Capacitors" deviceset="CAP" device="PTH"/>
@@
 <text x="166.116" y="115.316" size="1.778" layer="97">USER
 LED</text>
-<text x="167.64" y="7.62" size="3.81" layer="91">Mike Hord</text>
-<text x="238.76" y="6.096" size="3.81" layer="91">13</text>
+<text x="167.64" y="7.62" size="3.81" layer="94">Mike Hord</text>
+<text x="238.76" y="6.096" size="3.81" layer="94">14</text>
 </plain>
 <instances>
@@
 Caps</text>
 <text x="55.88" y="111.76" size="3.81" layer="97">Target Supply Pins</text>
-<wire x1="124.46" y1="109.22" x2="248.92" y2="109.22" width="0.3048" layer="94" style="longdash"/>
+<wire x1="124.46" y1="109.22" x2="248.92" y2="109.22" width="0.3048" layer="97" style="longdash"/>
 <wire x1="121.92" y1="185.42" x2="124.46" y2="185.42" width="0.3048" layer="94" style="longdash"/>
 <wire x1="124.46" y1="185.42" x2="124.46" y2="109.22" width="0.3048" layer="97" style="longdash"/>
@@
 battery operation</text>
 <text x="35.56" y="17.78" size="1.778" layer="97">JP3 is DNP</text>
-<text x="167.64" y="7.62" size="3.81" layer="91">Mike Hord</text>
-<text x="238.252" y="6.096" size="3.81" layer="91">13</text>
+<text x="167.64" y="7.62" size="3.81" layer="94">Mike Hord</text>
+<text x="238.252" y="6.096" size="3.81" layer="94">14</text>
 <text x="121.92" y="33.528" size="0.6096" layer="97">C37 &amp; C38 to be
 near U2 &amp;U 3 input</text>
@@
 </instance>
 <instance part="SUPPLY3" gate="G$1" x="50.8" y="179.07"/>
-<instance part="GND5" gate="1" x="17.78" y="60.96"/>
 <instance part="C26" gate="G$1" x="185.42" y="50.8" rot="R180"/>
 <instance part="C28" gate="G$1" x="198.12" y="50.8" rot="R180"/>
@@
 </segment>
 <segment>
-<pinref part="GND5" gate="1" pin="GND"/>
-<wire x1="17.78" y1="63.5" x2="17.78" y2="68.58" width="0.1524" layer="91"/>
-<pinref part="JP1" gate="G$1" pin="SHIELD"/>
-<wire x1="17.78" y1="68.58" x2="17.78" y2="91.44" width="0.1524" layer="91"/>
-<wire x1="17.78" y1="91.44" x2="33.02" y2="91.44" width="0.1524" layer="91"/>
-<pinref part="JP2" gate="G$1" pin="SHIELD"/>
-<wire x1="33.02" y1="68.58" x2="17.78" y2="68.58" width="0.1524" layer="91"/>
-<junction x="17.78" y="68.58"/>
-</segment>
-<segment>
 <pinref part="GND34" gate="1" pin="GND"/>
 <pinref part="C26" gate="G$1" pin="1"/>
@@
 <pinref part="R12" gate="G$1" pin="1"/>
 <wire x1="198.12" y1="53.34" x2="198.12" y2="55.88" width="0.1524" layer="91"/>
+</segment>
+</net>
+<net name="ANCHOR_POUR" class="0">
+<segment>
+<pinref part="JP1" gate="G$1" pin="SHIELD"/>
+<wire x1="25.4" y1="68.58" x2="25.4" y2="91.44" width="0.1524" layer="91"/>
+<wire x1="25.4" y1="91.44" x2="33.02" y2="91.44" width="0.1524" layer="91"/>
+<pinref part="JP2" gate="G$1" pin="SHIELD"/>
+<wire x1="33.02" y1="68.58" x2="25.4" y2="68.58" width="0.1524" layer="91"/>
+<wire x1="25.4" y1="91.44" x2="22.86" y2="91.44" width="0.1524" layer="91"/>
+<junction x="25.4" y="91.44"/>
+<label x="22.86" y="91.44" size="1.778" layer="95" rot="R180" xref="yes"/>
 </segment>
 </net>
@@
 Close to connect debugger
 to target via I2C</text>
-<text x="167.64" y="7.62" size="3.81" layer="91">Mike Hord</text>
-<text x="237.744" y="6.35" size="3.81" layer="91">13</text>
+<text x="167.64" y="7.62" size="3.81" layer="94">Mike Hord</text>
+<text x="237.744" y="6.35" size="3.81" layer="94">14</text>
 </plain>
 <instances>
